File: TemperatureHumidityEPD.kicad_pcb (KiCad board)
At the start: 2 copper layers, 0 parts

Commit message: PCB Design
Parts:
- added BT1: Battery_Cell, KevinLibrary:CR2032_BATTERY_HOLDER, B.Cu at (124.0, 96.5)
- added C1: 100n, Capacitors_SMD:C_0805_HandSoldering, F.Cu at (114.1, 92.0)
- added C2: 100n, Capacitors_SMD:C_0805_HandSoldering, F.Cu at (114.1, 97.6)
- added C3: 100n, Capacitors_SMD:C_0805_HandSoldering, F.Cu at (126.7, 96.9)
- added C4: 10u, Capacitors_SMD:C_0805_HandSoldering, F.Cu at (128.5, 85.0)
- added C5: 100n, Capacitors_SMD:C_0805_HandSoldering, F.Cu at (135.4, 99.3)
- added J1: Conn_01x08, Pin_Headers:Pin_Header_Straight_1x08_Pitch2.54mm, F.Cu at (102.8, 105.9)
- added J2: Conn_01x05, Pin_Headers:Pin_Header_Straight_1x05_Pitch2.54mm, F.Cu at (145.2, 91.8)
- added J3: Conn_01x02, Pin_Headers:Pin_Header_Straight_1x02_Pitch2.54mm, F.Cu at (134.0, 85.0)
- added L1: 600Ohm, Resistors_SMD:R_0805_HandSoldering, F.Cu at (116.3, 103.0)
- added MP1: MOUNTHOLE, KevinLibrary:TH-M3, F.Cu at (145.5, 110.5)
- added MP2: MOUNTHOLE, KevinLibrary:TH-M3, F.Cu at (102.5, 82.5)
- added MP3: MOUNTHOLE, KevinLibrary:TH-M3, F.Cu at (102.5, 110.5)
- added MP4: MOUNTHOLE, KevinLibrary:TH-M3, F.Cu at (145.5, 82.5)
- added R1: 10K, Resistors_SMD:R_0805_HandSoldering, F.Cu at (118.8, 90.5)
- added R2: 10K, Resistors_SMD:R_0805_HandSoldering, F.Cu at (130.2, 91.1)
- added R3: 10K, Resistors_SMD:R_0805_HandSoldering, F.Cu at (133.4, 91.0)
- added REF**: VIA_13MIL, KevinLibrary:VIA_13MIL, F.Cu at (128.3, 94.5)
- added REF**: VIA_13MIL, KevinLibrary:VIA_13MIL, F.Cu at (123.6, 102.0)
- added REF**: Logo, KevinLibrary:Logo, F.Cu at (136.7, 108.3)
- added U1: STM32L031Fx, Housings_SSOP:TSSOP-20_4.4x6.5mm_Pitch0.65mm, F.Cu at (120.3, 96.6)
- added U2: SI7021, KevinLibrary:SI7021, F.Cu at (131.6, 96.6)
Routing:
- net +3V3: track 0.00 -> 125.6 mm
- net /NRST: track 0.00 -> 42.5 mm, vias 0 -> 1
- net /SCK: track 0.00 -> 34.2 mm
- net /MOSI: track 0.00 -> 32.4 mm
- net /SWCLK: track 0.00 -> 30.2 mm, vias 0 -> 1
- net /SWDIO: track 0.00 -> 24.8 mm, vias 0 -> 1
- net /BUSY: track 0.00 -> 17.5 mm
- net /RST: track 0.00 -> 16.4 mm
- net /SCL: track 0.00 -> 15.8 mm
- net /DC: track 0.00 -> 15.8 mm
- net /SPI_CS: track 0.00 -> 14.8 mm
- net /SDA: track 0.00 -> 11.4 mm, vias 0 -> 2
- net Net-(C2-Pad1): track 0.00 -> 11.4 mm
- net Net-(R1-Pad1): track 0.00 -> 4.40 mm
- net GND: track 0.00 -> 2.88 mm
- added copper zone on B.Cu, net GND
- added copper zone on F.Cu, net GND
Other:
- board outline added: 48 x 33 mm
- net class Default: clearance 0.254 -> 0.1524
- net class Power added: clearance 0.3048, trace_width 0.3048, via_dia 0.6858, via_drill 0.3302
- rule trace_clearance: 0.254 -> 0.1524
- board text added: "Kevin Kessler 2018"
