File: TemperatureHumidityEPD.kicad_pcb (KiCad board)
At the start: 2 copper layers, 48 x 33 mm, 22 parts, among them J1 Conn_01x08, J2 Conn_01x05, J3 Conn_01x02, U1 STM32L031Fx, U2 SI7021

Commit message: Switching Transistor
Parts:
- added Q1: IRLML6344, TO_SOT_Packages_SMD:SOT-23, F.Cu at (112.8, 84.2)
- added R4: 100R, Resistors_SMD:R_0805_HandSoldering, F.Cu at (118.9, 83.0)
- added R5: 100K, Resistors_SMD:R_0805_HandSoldering, F.Cu at (118.9, 85.8)
Connections:
- J1 pad 7: GND -> /EPD_GND
- U1 pad 12: (no net) -> /EPD_POWER
- U1 pad 14: (no net) -> GND
- U1 pad 2: (no net) -> GND
- U1 pad 3: (no net) -> GND
- U1 pad 6: (no net) -> GND
Routing:
- net /EPD_POWER: track 0.00 -> 23.5 mm, vias 0 -> 2
- net /EPD_GND: track 0.00 -> 11.7 mm
- net Net-(Q1-Pad1): track 0.00 -> 6.85 mm
