File: TemperatureHumidityEPD.sch (KiCad schematic (older format))
At the start: 5 parts

Commit message: Schematic
Parts:
- added BT?: Battery_Cell, symbol Battery_Cell
- added C?: 10u, symbol C
- added C? (x2): 100n, symbol C
- added J?: Conn_01x08, symbol Conn_01x08
- added J?: Conn_01x05, symbol Conn_01x05
- added R?: R, symbol R
Connections:
- net labels added: +3V3, BUSY, DC, GND, MOSI, RST, SCK, SCL, SDA, SPI_CS, SWCLK, SWDIO
- wire segments 0 -> 51
Other:
- moved on the sheet: R?

Commit message: PCB Design
Parts:
- added C3, C5: 100n, Capacitors_SMD:C_0805_HandSoldering, symbol C
- added L1: 600Ohm, Resistors_SMD:R_0805_HandSoldering, symbol L_Core_Ferrite_Small
- added MP1, MP2, MP3, MP4: MOUNTHOLE, KevinLibrary:TH-M3, symbol MOUNTHOLE
- BT1: renamed from BT?; footprint (none) -> KevinLibrary:CR2032_BATTERY_HOLDER
- C1, C2, C4: renamed from C?; footprint (none) -> Capacitors_SMD:C_0805_HandSoldering
- J1: renamed from J?; footprint (none) -> Pin_Headers:Pin_Header_Straight_1x08_Pitch2.54mm
- J2: renamed from J?; footprint (none) -> Pin_Headers:Pin_Header_Straight_1x05_Pitch2.54mm
- J3: renamed from J?; footprint (none) -> Pin_Headers:Pin_Header_Straight_1x02_Pitch2.54mm
- R1, R2, R3: renamed from R?; value R -> 10K; footprint (none) -> Resistors_SMD:R_0805_HandSoldering
- U1: renamed from U?; footprint MODULE -> Housings_SSOP:TSSOP-20_4.4x6.5mm_Pitch0.65mm
- U2: renamed from U?; footprint MODULE -> KevinLibrary:SI7021
Connections:
- net labels added: NRST
- wire segments 51 -> 76
- no-connect marks 0 -> 5
Other:
- moved on the sheet: C2

Commit message: Switching Transistor
Parts:
- added Q1: IRLML6344, TO_SOT_Packages_SMD:SOT-23, symbol IRLML6344
- added R4: 100R, Resistors_SMD:R_0805_HandSoldering, symbol R
- added R5: 100K, Resistors_SMD:R_0805_HandSoldering, symbol R
Connections:
- net labels added: EPD_GND, EPD_POWER
- wire segments 76 -> 89
- no-connect marks 5 -> 0
Changed lines of the file:
@@
 	6250 1850 7150 1850
 Connection ~ 6450 1850
-$Comp
-L PWR_FLAG #FLG04
-U 1 1 5ACA9F25
-P 6200 2200
-F 0 "#FLG04" H 6200 2275 50  0001 C CNN
-F 1 "PWR_FLAG" H 6200 2350 50  0000 C CNN
-F 2 "" H 6200 2200 50  0001 C CNN
-F 3 "" H 6200 2200 50  0001 C CNN
-	1    6200 2200
-	1    0    0    -1
-$EndComp
 Wire Wire Line
 	6200 2200 6200 2250
@@
 Connection ~ 6450 2250
 $Comp
-L +3V3 #PWR05
+L +3V3 #PWR04
 U 1 1 5ACA9F54
 P 7650 2150
-F 0 "#PWR05" H 7650 2000 50  0001 C CNN
+F 0 "#PWR04" H 7650 2000 50  0001 C CNN
 F 1 "+3V3" H 7650 2290 50  0000 C CNN
 F 2 "" H 7650 2150 50  0001 C CNN
@@
 $EndComp
 $Comp
-L GND #PWR06
+L GND #PWR05
 U 1 1 5ACA9F74
 P 7650 2350
-F 0 "#PWR06" H 7650 2100 50  0001 C CNN
+F 0 "#PWR05" H 7650 2100 50  0001 C CNN
 F 1 "GND" H 7650 2200 50  0000 C CNN
 F 2 "" H 7650 2350 50  0001 C CNN
@@
 	7650 2300 7650 2350
 $Comp
-L +3V3 #PWR07
+L +3V3 #PWR06
 U 1 1 5ACA9FF6
 P 6700 3000
-F 0 "#PWR07" H 6700 2850 50  0001 C CNN
+F 0 "#PWR06" H 6700 2850 50  0001 C CNN
 F 1 "+3V3" H 6700 3140 50  0000 C CNN
 F 2 "" H 6700 3000 50  0001 C CNN
@@
 $EndComp
 $Comp
-L +3V3 #PWR08
+L +3V3 #PWR07
 U 1 1 5ACAA016
 P 8700 3000
-F 0 "#PWR08" H 8700 2850 50  0001 C CNN
+F 0 "#PWR07" H 8700 2850 50  0001 C CNN
 F 1 "+3V3" H 8700 3140 50  0000 C CNN
 F 2 "" H 8700 3000 50  0001 C CNN
@@
 	4500 2200 4200 2200
 $Comp
-L +3V3 #PWR09
+L +3V3 #PWR08
 U 1 1 5ACAA39E
 P 4100 2400
-F 0 "#PWR09" H 4100 2250 50  0001 C CNN
+F 0 "#PWR08" H 4100 2250 50  0001 C CNN
 F 1 "+3V3" H 4100 2540 50  0000 C CNN
 F 2 "" H 4100 2400 50  0001 C CNN
@@
 $EndComp
 $Comp
-L GND #PWR010
+L GND #PWR09
 U 1 1 5ACAA3C4
-P 4300 2350
-F 0 "#PWR010" H 4300 2100 50  0001 C CNN
-F 1 "GND" H 4300 2200 50  0000 C CNN
-F 2 "" H 4300 2350 50  0001 C CNN
-F 3 "" H 4300 2350 50  0001 C CNN
-	1    4300 2350
+P 7500 5000
+F 0 "#PWR09" H 7500 4750 50  0001 C CNN
+F 1 "GND" H 7500 4850 50  0000 C CNN
+F 2 "" H 7500 5000 50  0001 C CNN
+F 3 "" H 7500 5000 50  0001 C CNN
+	1    7500 5000
 	1    0    0    -1
 $EndComp
@@
 MOSI
 $Comp
-L +3V3 #PWR011
+L +3V3 #PWR010
 U 1 1 5ACAA802
 P 3650 3450
-F 0 "#PWR011" H 3650 3300 50  0001 C CNN
+F 0 "#PWR010" H 3650 3300 50  0001 C CNN
 F 1 "+3V3" H 3650 3590 50  0000 C CNN
 F 2 "" H 3650 3450 50  0001 C CNN
@@
 $EndComp
 $Comp
-L GND #PWR012
+L GND #PWR011
 U 1 1 5ACAA828
 P 3650 4200
-F 0 "#PWR012" H 3650 3950 50  0001 C CNN
+F 0 "#PWR011" H 3650 3950 50  0001 C CNN
 F 1 "GND" H 3650 4050 50  0000 C CNN
 F 2 "" H 3650 4200 50  0001 C CNN
@@
 $EndComp
 $Comp
-L GND #PWR013
+L GND #PWR012
 U 1 1 5ACAAB96
 P 3200 3500
-F 0 "#PWR013" H 3200 3250 50  0001 C CNN
+F 0 "#PWR012" H 3200 3250 50  0001 C CNN
 F 1 "GND" H 3200 3350 50  0000 C CNN
 F 2 "" H 3200 3500 50  0001 C CNN
@@
 $EndComp
 $Comp
-L +3V3 #PWR014
+L +3V3 #PWR013
 U 1 1 5ACAB389
 P 8950 3400
-F 0 "#PWR014" H 8950 3250 50  0001 C CNN
+F 0 "#PWR013" H 8950 3250 50  0001 C CNN
 F 1 "+3V3" H 8950 3540 50  0000 C CNN
 F 2 "" H 8950 3400 50  0001 C CNN
@@
 $EndComp
 $Comp
-L GND #PWR015
+L GND #PWR014
 U 1 1 5ACAB3B8
 P 6750 3650
-F 0 "#PWR015" H 6750 3400 50  0001 C CNN
+F 0 "#PWR014" H 6750 3400 50  0001 C CNN
 F 1 "GND" H 6750 3500 50  0000 C CNN
 F 2 "" H 6750 3650 50  0001 C CNN
@@
 $EndComp
 $Comp
-L +3V3 #PWR016
+L +3V3 #PWR015
 U 1 1 5ACAB447
 P 6350 3250
-F 0 "#PWR016" H 6350 3100 50  0001 C CNN
+F 0 "#PWR015" H 6350 3100 50  0001 C CNN
 F 1 "+3V3" H 6350 3390 50  0000 C CNN
 F 2 "" H 6350 3250 50  0001 C CNN
@@
 $EndComp
 $Comp
-L GND #PWR017
+L GND #PWR016
 U 1 1 5ACAB479
 P 6350 3900
-F 0 "#PWR017" H 6350 3650 50  0001 C CNN
+F 0 "#PWR016" H 6350 3650 50  0001 C CNN
 F 1 "GND" H 6350 3750 50  0000 C CNN
 F 2 "" H 6350 3900 50  0001 C CNN
@@
 $EndComp
 $Comp
-L GND #PWR018
+L GND #PWR017
 U 1 1 5ACAB846
 P 8950 4000
-F 0 "#PWR018" H 8950 3750 50  0001 C CNN
+F 0 "#PWR017" H 8950 3750 50  0001 C CNN
 F 1 "GND" H 8950 3850 50  0000 C CNN
 F 2 "" H 8950 4000 50  0001 C CNN
@@
 SWCLK
 $Comp
-L +3V3 #PWR019
+L +3V3 #PWR018
 U 1 1 5ACABE7A
 P 5000 1650
-F 0 "#PWR019" H 5000 1500 50  0001 C CNN
+F 0 "#PWR018" H 5000 1500 50  0001 C CNN
 F 1 "+3V3" H 5000 1790 50  0000 C CNN
 F 2 "" H 5000 1650 50  0001 C CNN
@@
 	5000 1750 5000 1650
 $Comp
-L GND #PWR020
+L GND #PWR019
 U 1 1 5ACABF0A
 P 4900 2100
-F 0 "#PWR020" H 4900 1850 50  0001 C CNN
+F 0 "#PWR019" H 4900 1850 50  0001 C CNN
 F 1 "GND" H 4900 1950 50  0000 C CNN
 F 2 "" H 4900 2100 50  0001 C CNN
@@
 	3800 3750 3350 3750
 Connection ~ 3650 3750
-NoConn ~ 4200 3200
-NoConn ~ 4200 3300
-NoConn ~ 4200 3600
-NoConn ~ 5700 3700
-NoConn ~ 5700 3900
-$Comp
-L PWR_FLAG #FLG021
+$Comp
+L PWR_FLAG #FLG020
 U 1 1 5ACAD3B1
 P 3350 3800
-F 0 "#FLG021" H 3350 3875 50  0001 C CNN
+F 0 "#FLG020" H 3350 3875 50  0001 C CNN
 F 1 "PWR_FLAG" H 3350 3950 50  0000 C CNN
 F 2 "" H 3350 3800 50  0001 C CNN
@@
 $EndComp
 Wire Wire Line
-	4500 2300 4300 2300
-Wire Wire Line
-	4300 2300 4300 2350
+	4500 2300 4200 2300
 Wire Wire Line
 	4500 2400 4400 2400
@@
 Wire Wire Line
 	4100 2600 4100 2400
+Wire Wire Line
+	5700 3900 6100 3900
+Text Label 5700 3900 0    60   ~ 0
+EPD_POWER
+Text Label 4200 2300 0    60   ~ 0
+EPD_GND
+$Comp
+L IRLML6344 Q1
+U 1 1 5B11E118
+P 7400 4450
+F 0 "Q1" H 7600 4525 50  0000 L CNN
+F 1 "IRLML6344" H 7600 4450 50  0000 L CNN
+F 2 "TO_SOT_Packages_SMD:SOT-23" H 7600 4375 50  0001 L CIN
+F 3 "" H 7400 4450 50  0000 L CNN
+	1    7400 4450
+	1    0    0    -1
+$EndComp
+Wire Wire Line
+	7500 4650 7500 5000
+$Comp
+L R R4
+U 1 1 5B11E229
+P 6850 4500
+F 0 "R4" V 6930 4500 50  0000 C CNN
+F 1 "100R" V 6850 4500 50  0000 C CNN
+F 2 "Resistors_SMD:R_0805_HandSoldering" V 6780 4500 50  0001 C CNN
+F 3 "" H 6850 4500 50  0001 C CNN
+	1    6850 4500
+	0    1    1    0
+$EndComp
+$Comp
+L R R5
+U 1 1 5B11E296
+P 7100 4700
+F 0 "R5" V 7180 4700 50  0000 C CNN
+F 1 "100K" V 7100 4700 50  0000 C CNN
+F 2 "Resistors_SMD:R_0805_HandSoldering" V 7030 4700 50  0001 C CNN
+F 3 "" H 7100 4700 50  0001 C CNN
+	1    7100 4700
+	-1   0    0    1
+$EndComp
+Wire Wire Line
+	7100 4850 7100 4900
+Wire Wire Line
+	7100 4900 7500 4900
+Connection ~ 7500 4900
+Wire Wire Line
+	7000 4500 7200 4500
+Wire Wire Line
+	7100 4550 7100 4500
+Connection ~ 7100 4500
+Wire Wire Line
+	6700 4500 6200 4500
+Wire Wire Line
+	7500 4250 7500 4150
+Wire Wire Line
+	7500 4150 7900 4150
+Text Label 6200 4500 0    60   ~ 0
+EPD_POWER
+Text Label 7500 4150 0    60   ~ 0
+EPD_GND
+Wire Wire Line
+	5700 3700 6100 3700
+Text Label 5800 3700 0    60   ~ 0
+GND
+Wire Wire Line
+	4200 3600 3900 3600
+Text Label 3950 3600 0    60   ~ 0
+GND
+Wire Wire Line
+	4200 3200 3950 3200
+Wire Wire Line
+	4200 3300 4100 3300
+Wire Wire Line
+	4100 3300 4100 3200
+Connection ~ 4100 3200
+Text Label 3950 3200 0    60   ~ 0
+GND
 $EndSCHEMATC
